Commit message: 修复bug，在wsl运行

File: ackermann_gazebo_sim/src/racebot_description/urdf/ackermann/racecar.xacro (robot description, xacro)
@@ -1,4 +1,6 @@
 <?xml version="1.0" encoding="utf-8"?>
 <robot name="racebot" xmlns:xacro="http://www.ros.org/wiki/xacro">
+    <xacro:arg name="robot_name" default="racebot"/>
+    <xacro:property name="robot_name" value="$(arg robot_name)"/>
     <xacro:include filename="$(find racebot_description)/urdf/ackermann/macros.xacro" />
     <link name="base_footprint">
